File: Rev_2/ECAD/board/Kicad/EEPROM_PROGRAMMER.kicad_pcb (KiCad board)
At the start: 4 copper layers, 0 parts

Commit message: Added missing 3D-models aswell as fixed wrong footprints
Parts:
- added C1: 100u, Capacitor_THT:CP_Radial_D6.3mm_P2.50mm, F.Cu at (-93.9, 79.7)
- added C10: 22p, Capacitor_SMD:C_0805_2012Metric_Pad1.18x1.45mm_HandSolder, F.Cu at (-69.9, 79.7)
- added C101: 100n, Capacitor_SMD:C_0805_2012Metric_Pad1.18x1.45mm_HandSolder, F.Cu at (-60.3, 28.2)
- added C102: 100n, Capacitor_SMD:C_0805_2012Metric_Pad1.18x1.45mm_HandSolder, F.Cu at (-60.3, 36.0)
- added C103: 100n, Capacitor_SMD:C_0805_2012Metric_Pad1.18x1.45mm_HandSolder, F.Cu at (-52.4, 28.2)
- added C104: 100n, Capacitor_SMD:C_0805_2012Metric_Pad1.18x1.45mm_HandSolder, F.Cu at (-52.4, 36.0)
- added C105: 100n, Capacitor_SMD:C_0805_2012Metric_Pad1.18x1.45mm_HandSolder, F.Cu at (-44.4, 28.2)
- added C106: 4u7, Capacitor_SMD:C_0805_2012Metric_Pad1.18x1.45mm_HandSolder, F.Cu at (-44.4, 36.0)
- added C107: 1u, Capacitor_SMD:C_0805_2012Metric_Pad1.18x1.45mm_HandSolder, F.Cu at (-36.4, 28.2)
- added C108: 100n, Capacitor_SMD:C_0805_2012Metric_Pad1.18x1.45mm_HandSolder, F.Cu at (-36.4, 36.0)
- added C11: 22p, Capacitor_SMD:C_0805_2012Metric_Pad1.18x1.45mm_HandSolder, F.Cu at (-69.9, 87.6)
- added C12: 100n, Capacitor_SMD:C_0805_2012Metric_Pad1.18x1.45mm_HandSolder, F.Cu at (-69.9, 95.4)
- added C2: 100n, Capacitor_SMD:C_0805_2012Metric_Pad1.18x1.45mm_HandSolder, F.Cu at (-93.9, 87.6)
- added C3: 100u, Capacitor_THT:CP_Radial_D6.3mm_P2.50mm, F.Cu at (-93.9, 95.4)
- added C4: 100n, Capacitor_SMD:C_0805_2012Metric_Pad1.18x1.45mm_HandSolder, F.Cu at (-85.9, 79.7)
- added C5: 4u7, Capacitor_SMD:C_0805_2012Metric_Pad1.18x1.45mm_HandSolder, F.Cu at (-85.9, 87.6)
- added C6: 100n, Capacitor_SMD:C_0805_2012Metric_Pad1.18x1.45mm_HandSolder, F.Cu at (-85.9, 95.4)
- added C7: 100n, Capacitor_SMD:C_0805_2012Metric_Pad1.18x1.45mm_HandSolder, F.Cu at (-77.9, 79.7)
- added C8: 100n, Capacitor_SMD:C_0805_2012Metric_Pad1.18x1.45mm_HandSolder, F.Cu at (-77.9, 87.6)
- added C9: 100n, Capacitor_SMD:C_0805_2012Metric_Pad1.18x1.45mm_HandSolder, F.Cu at (-77.9, 95.4)
- added D1: RED, LED_SMD:LED_0805_2012Metric_Pad1.15x1.40mm_HandSolder, F.Cu at (-57.3, 88.3)
- added D101: BLUE, LED_SMD:LED_0805_2012Metric_Pad1.15x1.40mm_HandSolder, F.Cu at (-36.5, 41.5)
- added D102: BLUE, LED_SMD:LED_0805_2012Metric_Pad1.15x1.40mm_HandSolder, F.Cu at (-36.5, 44.5)
- added D103: BLUE, LED_SMD:LED_0805_2012Metric_Pad1.15x1.40mm_HandSolder, F.Cu at (-36.5, 47.5)
- added D104: BLUE, LED_SMD:LED_0805_2012Metric_Pad1.15x1.40mm_HandSolder, F.Cu at (-36.5, 50.6)
- added D105: BLUE, LED_SMD:LED_0805_2012Metric_Pad1.15x1.40mm_HandSolder, F.Cu at (-36.5, 53.6)
- added D106: BLUE, LED_SMD:LED_0805_2012Metric_Pad1.15x1.40mm_HandSolder, F.Cu at (-36.5, 56.6)
- added D107: BLUE, LED_SMD:LED_0805_2012Metric_Pad1.15x1.40mm_HandSolder, F.Cu at (-36.5, 59.7)
- added D108: BLUE, LED_SMD:LED_0805_2012Metric_Pad1.15x1.40mm_HandSolder, F.Cu at (-31.8, 41.5)
- added D109: BLUE, LED_SMD:LED_0805_2012Metric_Pad1.15x1.40mm_HandSolder, F.Cu at (-31.8, 44.5)
- added D110: BLUE, LED_SMD:LED_0805_2012Metric_Pad1.15x1.40mm_HandSolder, F.Cu at (-31.8, 47.5)
- added D111: BLUE, LED_SMD:LED_0805_2012Metric_Pad1.15x1.40mm_HandSolder, F.Cu at (-31.8, 50.6)
- added D112: BLUE, LED_SMD:LED_0805_2012Metric_Pad1.15x1.40mm_HandSolder, F.Cu at (-31.8, 53.6)
- added D113: BLUE, LED_SMD:LED_0805_2012Metric_Pad1.15x1.40mm_HandSolder, F.Cu at (-31.8, 56.6)
- added D114: GREEN, LED_SMD:LED_0805_2012Metric_Pad1.15x1.40mm_HandSolder, F.Cu at (-31.8, 59.7)
- added D115: GREEN, LED_SMD:LED_0805_2012Metric_Pad1.15x1.40mm_HandSolder, F.Cu at (-27.0, 41.5)
- added D116: GREEN, LED_SMD:LED_0805_2012Metric_Pad1.15x1.40mm_HandSolder, F.Cu at (-27.0, 44.5)
- added D117: GREEN, LED_SMD:LED_0805_2012Metric_Pad1.15x1.40mm_HandSolder, F.Cu at (-27.0, 47.5)
- added D118: GREEN, LED_SMD:LED_0805_2012Metric_Pad1.15x1.40mm_HandSolder, F.Cu at (-27.0, 50.6)
- added D119: GREEN, LED_SMD:LED_0805_2012Metric_Pad1.15x1.40mm_HandSolder, F.Cu at (-27.0, 53.6)
- added D120: GREEN, LED_SMD:LED_0805_2012Metric_Pad1.15x1.40mm_HandSolder, F.Cu at (-27.0, 56.6)
- added D121: GREEN, LED_SMD:LED_0805_2012Metric_Pad1.15x1.40mm_HandSolder, F.Cu at (-27.0, 59.7)
- added D2: 9V, Diode_THT:D_DO-35_SOD27_P3.81mm_Vertical_AnodeUp, F.Cu at (-59.9, 116.3)
- added D5: READ, LED_SMD:LED_0805_2012Metric_Pad1.15x1.40mm_HandSolder, F.Cu at (-57.3, 91.4)
- added D6: WRITE, LED_SMD:LED_0805_2012Metric_Pad1.15x1.40mm_HandSolder, F.Cu at (-57.3, 94.4)
- added JP1: Jumper, Jumper:SolderJumper-2_P1.3mm_Open_TrianglePad1.0x1.5mm, F.Cu at (-59.7, 120.0)
- added Q1: PMOS, Package_TO_SOT_SMD:SOT-23, F.Cu at (-59.4, 107.8)
- added Q4: NPN, Package_TO_SOT_SMD:SOT-23, F.Cu at (-59.4, 112.2)
- added R1: 4k7, Resistor_SMD:R_0805_2012Metric_Pad1.20x1.40mm_HandSolder, F.Cu at (-94.3, 100.8)
- added R10: 4k7, Resistor_SMD:R_0805_2012Metric_Pad1.20x1.40mm_HandSolder, F.Cu at (-94.3, 115.6)
- added R101: 10k, Resistor_SMD:R_0805_2012Metric_Pad1.20x1.40mm_HandSolder, F.Cu at (-50.8, 41.4)
- added R102: 10k, Resistor_SMD:R_0805_2012Metric_Pad1.20x1.40mm_HandSolder, F.Cu at (-50.8, 44.4)
- added R103: 4k7, Resistor_SMD:R_0805_2012Metric_Pad1.20x1.40mm_HandSolder, F.Cu at (-50.8, 47.3)
- added R104: 4k7, Resistor_SMD:R_0805_2012Metric_Pad1.20x1.40mm_HandSolder, F.Cu at (-50.8, 50.3)
- added R105: 4k7, Resistor_SMD:R_0805_2012Metric_Pad1.20x1.40mm_HandSolder, F.Cu at (-50.8, 53.2)
- added R106: 4k7, Resistor_SMD:R_0805_2012Metric_Pad1.20x1.40mm_HandSolder, F.Cu at (-50.8, 56.2)
- added R107: 4k7, Resistor_SMD:R_0805_2012Metric_Pad1.20x1.40mm_HandSolder, F.Cu at (-50.8, 59.1)
- added R108: 4k7, Resistor_SMD:R_0805_2012Metric_Pad1.20x1.40mm_HandSolder, F.Cu at (-50.8, 62.1)
- added R109: 4k7, Resistor_SMD:R_0805_2012Metric_Pad1.20x1.40mm_HandSolder, F.Cu at (-46.1, 41.4)
- added R11: 10k, Resistor_SMD:R_0805_2012Metric_Pad1.20x1.40mm_HandSolder, F.Cu at (-94.3, 118.5)
- added R110: 4k7, Resistor_SMD:R_0805_2012Metric_Pad1.20x1.40mm_HandSolder, F.Cu at (-46.1, 44.4)
- added R111: 4k7, Resistor_SMD:R_0805_2012Metric_Pad1.20x1.40mm_HandSolder, F.Cu at (-46.1, 47.3)
- added R112: 4k7, Resistor_SMD:R_0805_2012Metric_Pad1.20x1.40mm_HandSolder, F.Cu at (-46.1, 50.3)
- added R113: 4k7, Resistor_SMD:R_0805_2012Metric_Pad1.20x1.40mm_HandSolder, F.Cu at (-46.1, 53.2)
- added R114: 4k7, Resistor_SMD:R_0805_2012Metric_Pad1.20x1.40mm_HandSolder, F.Cu at (-46.1, 56.2)
- added R115: 4k7, Resistor_SMD:R_0805_2012Metric_Pad1.20x1.40mm_HandSolder, F.Cu at (-46.1, 59.1)
- added R116: 4k7, Resistor_SMD:R_0805_2012Metric_Pad1.20x1.40mm_HandSolder, F.Cu at (-46.1, 62.1)
- added R117: 4k7, Resistor_SMD:R_0805_2012Metric_Pad1.20x1.40mm_HandSolder, F.Cu at (-41.3, 41.4)
- added R118: 4k7, Resistor_SMD:R_0805_2012Metric_Pad1.20x1.40mm_HandSolder, F.Cu at (-41.3, 44.4)
- added R119: 4k7, Resistor_SMD:R_0805_2012Metric_Pad1.20x1.40mm_HandSolder, F.Cu at (-41.3, 47.3)
- added R120: 4k7, Resistor_SMD:R_0805_2012Metric_Pad1.20x1.40mm_HandSolder, F.Cu at (-41.3, 50.3)
- added R121: 4k7, Resistor_SMD:R_0805_2012Metric_Pad1.20x1.40mm_HandSolder, F.Cu at (-41.3, 53.2)
- added R122: 4k7, Resistor_SMD:R_0805_2012Metric_Pad1.20x1.40mm_HandSolder, F.Cu at (-41.3, 56.2)
- added R123: 4k7, Resistor_SMD:R_0805_2012Metric_Pad1.20x1.40mm_HandSolder, F.Cu at (-41.3, 59.1)
- added R13: 10k, Resistor_SMD:R_0805_2012Metric_Pad1.20x1.40mm_HandSolder, F.Cu at (-94.3, 121.5)
- added R2: 4k7, Resistor_SMD:R_0805_2012Metric_Pad1.20x1.40mm_HandSolder, F.Cu at (-94.3, 103.8)
- added R7: 10k, Resistor_SMD:R_0805_2012Metric_Pad1.20x1.40mm_HandSolder, F.Cu at (-94.3, 106.7)
- added R8: 10k, Resistor_SMD:R_0805_2012Metric_Pad1.20x1.40mm_HandSolder, F.Cu at (-94.3, 109.7)
- added R9: 4k7, Resistor_SMD:R_0805_2012Metric_Pad1.20x1.40mm_HandSolder, F.Cu at (-94.3, 112.6)
- added TP1: PWR, TestPoint:TestPoint_Keystone_5005-5009_Compact, F.Cu at (-62.2, 89.3)
- added TP2: GND, TestPoint:TestPoint_Keystone_5005-5009_Compact, F.Cu at (-62.2, 94.4)
- added U1: FT232RL, EEPROM_PROGRAMMER:FT232RL, F.Cu at (-83.4, 107.7)
- added U101: 4076B, EEPROM_PROGRAMMER:4076B, F.Cu at (-59.0, 18.0)
- added U102: 4076B, EEPROM_PROGRAMMER:4076B, F.Cu at (-50.8, 18.0)
- added U103: 4076B, EEPROM_PROGRAMMER:4076B, F.Cu at (-42.5, 18.0)
- added U104: 4076B, EEPROM_PROGRAMMER:4076B, F.Cu at (-34.3, 18.0)
- added U105: 74HC245, EEPROM_PROGRAMMER:74HC245, F.Cu at (-58.2, 53.8)
- added U106: AT28C64B-15PU, EEPROM_PROGRAMMER:AT28C64B-15PU, F.Cu at (-79.9, 67.3)
- added U2: ATMega328P-AU, EEPROM_PROGRAMMER:ATMega328P-AU, F.Cu at (-59.2, 81.3)
- added U3: ICSP, EEPROM_PROGRAMMER:ICSP, F.Cu at (-64.9, 102.5)
- added U4: SD_CARD_READER, EEPROM_PROGRAMMER:SD_CARD_READER, F.Cu at (-81.2, 102.5)
- added U5: SUM, EEPROM_PROGRAMMER:Summer, F.Cu at (-68.4, 112.1)
- added Y1: 16MHz, EEPROM_PROGRAMMER:Crystal, F.Cu at (-85.1, 114.2)

Commit message: Done with inital layout
Parts:
- added TP2: 5V, TestPoint:TestPoint_Keystone_5005-5009_Compact, F.Cu at (67.0, 44.5)
- moved R10 232.3 mm to (138.0, 115.0), turned to -90 degrees
- moved R9 229.3 mm to (135.0, 115.0), turned to 90 degrees
- moved U106 198.3 mm to (116.6, 93.5)
- moved D6 195.8 mm to (138.0, 109.0), turned to -90 degrees
- moved D5 193.1 mm to (135.0, 109.0), turned to 90 degrees
- moved R115 189.9 mm to (138.4, 104.1), turned to 90 degrees
- moved R114 187.2 mm to (134.9, 104.1), turned to 90 degrees
- moved R101 185.5 mm to (133.0, 66.0)
- moved R113 184.6 mm to (131.4, 104.1), turned to 90 degrees
- moved R112 182.1 mm to (127.9, 104.1), turned to 90 degrees
- moved R111 179.7 mm to (124.4, 104.1), turned to 90 degrees
- moved R110 177.4 mm to (120.9, 104.1), turned to 90 degrees
- moved C106 175.6 mm to (130.5, 51.5), turned to -90 degrees
- moved D113 175.4 mm to (138.4, 99.1), turned to -90 degrees
- moved R109 175.1 mm to (117.4, 104.1), turned to 90 degrees
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- renumbered TP2 to TP3
Connections:
- R1 pad 2: +5V -> GND
- R2 pad 2: +5V -> GND
Routing:
- net /POLARITY_PROTECTION: track 0.00 -> 17.1 mm
- net +5V: track 0.00 -> 13.9 mm
- net /VGS: track 0.00 -> 9.09 mm
- net /DTR: track 0.00 -> 5.27 mm
- net /RESET: track 0.00 -> 3.02 mm
- net Net-(D1-A): track 0.00 -> 1.98 mm
Other:
- board outline added: 100 x 83 mm
